File: STM32F407VET6/CoCo_Drive_Emulator.kicad_sch (KiCad schematic)
At the start: 7 parts, among them P1 CoCo_Slot, SW1 PB_Next, SW2 PB_Previous, U1 STM32F407VET6_DevBoard

Commit message: Added header for display
Parts:
- added J1: Conn_01x04, Connector_PinSocket_2.54mm:PinSocket_1x04_P2.54mm_Vertical, symbol Connector_Generic:Conn_01x04
Connections:
- net GND: now also J1.2 (Pin_2)
- net +3.3V: now reaches U1.3V3
- net +3.3V: now also J1.1 (Pin_1)
- net I2C3_SCL: now reaches U1.PA8
- net I2C3_SCL: now also J1.3 (Pin_3)
- net I2C3_SDA: now reaches U1.PC9
- net I2C3_SDA: now also J1.4 (Pin_4)
- no-connect marks 10 -> 8
